Commit message: files are configured to run with moveit

File: solid2ROS/urdf/robot_arm_urdf.urdf (robot description, URDF)
Before this commit: robot solid2ROS, 8 links, 7 joints
Joints:
- joint Joint_1: limit lower=0 upper=3.142 effort=300 velocity=3 -> lower=-3.142 upper=3.142 effort=300 velocity=3
- joint Joint_3: limit lower=0 upper=3.142 effort=200 velocity=3 -> lower=-3.142 upper=0 effort=200 velocity=3
- joint Joint_4: limit lower=0 upper=-3.142 effort=200 velocity=3 -> lower=-3.142 upper=0 effort=200 velocity=3
- joint Joint_6: limit lower=0 upper=-0.03 effort=100 velocity=3 -> lower=-0.03 upper=0.0 effort=100 velocity=3
